File: kicad_project/stripline_anode.kicad_pcb (KiCad board)
At the start: 6 copper layers, 244.9 x 347.7 mm, 104 parts, among them J1 QRM8-078-05.0-L-D-A, U1 anode_pad, U10 anode_pad, U11 anode_pad, U12 anode_pad, U13 anode_pad, U14 anode_pad, U15 anode_pad, U16 anode_pad, U17 anode_pad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

Commit message: Added logo silkscreen and footprint.
Parts:
- added G***: LOGO, logos:ellipse-logo, B.Cu at (279.0, 202.4)
Other:
- board text added: "LAPPD TOF FTBF Designers: Evan Angelico, Joe Pastika, Jacky Mengyang Li 2/2023, v2"
